File: petzki_6x13/kicad_petzki6x13/petzki6x13.kicad_pcb (KiCad board)
At the start: 2 copper layers, 150 parts

Commit message: Using TH-SMD diodes
Parts:
- D1, D10, D11, D12, D13, D14, D15, D16, D17, D18, D19, D2, D20, D21, D22, D23, D24, D25, D26, D27, D28, D29, D3, D30, D31, D32, D33, D34, D35, D36, D37, D38, D39, D4, D40, D41, D42, D43, D44, D45, D46, D47, D48, D49, D5, D50, D51, D52, D53, D54, D55, D56, D57, D58, D59, D6, D60, D61, D62, D63, D64, D65, D66, D67, D68, D69, D7, D70, D71, D72, D73, D74, D75, D8, D9: footprint ScottoKeebs_Components:Diode_SOD-123 -> Lily58-footprint:Diode_TH_SOD123
- moved D26 3.64 mm to (281.5, 63.0)
- moved D39 3.64 mm to (281.5, 82.1)
- moved D65 3.64 mm to (281.5, 120.2)
- moved D13 3.64 mm to (281.5, 44.0)
- moved D52 3.64 mm to (281.5, 101.1)
- moved D75 3.64 mm to (281.5, 139.2)
- moved D49 3.57 mm to (224.3, 101.1)
- moved D14 3.33 mm to (52.9, 63.0)
- moved D15 3.33 mm to (71.9, 63.0)
- moved D16 3.33 mm to (91.0, 63.0)
- moved D17 3.33 mm to (110.0, 63.0)
- moved D18 3.33 mm to (129.1, 63.0)
- moved D19 3.33 mm to (148.1, 63.0)
- moved D20 3.33 mm to (167.3, 63.0)
- moved D21 3.33 mm to (186.2, 63.0)
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Routing:
- net Net-(D53-K): track 227.1 -> 272.1 mm
- net Net-(D1-K): track 227.1 -> 272.1 mm
- net Net-(D40-K): track 227.1 -> 271.5 mm
- net Net-(D27-K): track 227.1 -> 271.5 mm
- net Net-(D14-K): track 227.1 -> 271.5 mm
- net Net-(D66-K): track 224.7 -> 259.8 mm
- net Net-(S22-Pad1): track 103.3 -> 100.2 mm, vias 10 -> 0
- net Net-(D49-A): track 8.99 -> 7.30 mm
- net Net-(D7-A): track 8.74 -> 7.30 mm
- net Net-(D70-A): track 8.74 -> 7.30 mm
- net Net-(D59-A): track 8.74 -> 7.30 mm
- net Net-(D5-A): track 8.74 -> 7.30 mm
- net Net-(D44-A): track 8.74 -> 7.30 mm
- net Net-(D31-A): track 8.74 -> 7.30 mm
- net Net-(D57-A): track 8.74 -> 7.30 mm
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
Commit message: added edge cut zone
Other:
- board outline added: 252.4 x 119.1 mm
Changed lines of the file:
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@@
       (net 49 "Net-(D46-A)") (pinfunction "A") (pintype "passive"))
   )
+  (gr_rect (start 31.42 31.63625) (end 283.8325 150.69875)
+    (stroke (width 0.1) (type default)) (fill none) (layer "Edge.Cuts"))
   (segment (start 262.40125 48.99621) (end 262.40379 48.99875) (width 0.25) (layer "F.Cu") (net 1))
   (segment (start 52.85125 45.69875) (end 52.85125 48.99621) (width 0.25) (layer "F.Cu") (net 1))
